File: pcb/nixie/nixie.sch (KiCad schematic (older format))
At the start: 21 parts, among them J2 Conn_01x02, P1 TTL_232R_3V3, Q1 Q_NMOS_DGS, U1 LM317EMP, U2 ESP-WROOM-32, U3 TACTILE, U4 TACTILE

Commit message: PCB work
Parts:
- added C9: 10u, Capacitor_SMD:C_2010_5025Metric, symbol Device:C
- added Q2, Q3, Q4: 2N7002, Package_TO_SOT_SMD:SOT-23, symbol myStuff:2N7002
- added R17, R18, R19: 1k, Resistor_SMD:R_0805_2012Metric, symbol Device:R
Connections:
- wire segments 94 -> 115

Commit message: Added MCP1630 idea
Parts:
- removed C5, C9: 10u, Capacitor_SMD:C_2010_5025Metric, symbol Device:C
- removed C6: 100n, Capacitor_SMD:C_0805_2012Metric, symbol Device:C
- removed D1: D, Diode_SMD:D_1206_3216Metric, symbol Device:D
- removed L1: L, myStuff:cc_5022, symbol Device:L
- removed Q1: Q_NMOS_DGS, Package_TO_SOT_SMD:SOT-23, symbol Device:Q_NMOS_DGS
- removed R2: 10R, Resistor_SMD:R_0805_2012Metric, symbol Device:R
- removed R5: 1M3, Resistor_SMD:R_0805_2012Metric, symbol Device:R
- removed R6: 7k15, Resistor_SMD:R_0805_2012Metric, symbol Device:R
- renumbered C1 to C?, C2 to C?, C4 to C?, C3 to C?, J2 to J?, P1 to P?, Q4 to Q?, Q3 to Q?, Q2 to Q?, R1 to R?, R3 to R?, R4 to R?, R17 to R?, R18 to R?, R19 to R?, U2 to U?, U1 to U?, U4 to U?, U3 to U?
Connections:
- net labels removed: HT
- wire segments 115 -> 91

Commit message: tricky
Parts:
- removed Q? (x3): 2N7002, Package_TO_SOT_SMD:SOT-23, symbol myStuff:2N7002
- removed R? (x3): 1k, Resistor_SMD:R_0805_2012Metric, symbol Device:R
- added J2: Conn_01x02, Connector_PinHeader_2.54mm:PinHeader_1x02_P2.54mm_Vertical, symbol Connector_Generic:Conn_01x02
- added U1: 74LVC3G34DP, Package_SO:VSSOP-8_2.4x2.1mm_P0.5mm, symbol myStuff:74LVC3G34DP
- C2: renamed from C?; value 470n -> 1u
- C3: renamed from C?; footprint Capacitor_SMD:C_2010_5025Metric -> Capacitor_SMD:C_1210_3225Metric
- gave numbers to parts that had none: 11
Connections:
- net labels added: HT, VCC
- net labels removed: +12V, vHtMon
- wire segments 91 -> 88
- no-connect marks 24 -> 25

Commit message: done, done done done
Parts:
- removed U1: 74LVC3G34DP, Package_SO:VSSOP-8_2.4x2.1mm_P0.5mm, symbol myStuff:74LVC3G34DP
- added C7: 1u, Capacitor_SMD:C_0805_2012Metric, symbol Device:C
- added J7: Conn_01x04, Connector_PinHeader_2.54mm:PinHeader_1x04_P2.54mm_Vertical, symbol Connector_Generic:Conn_01x04
- added U1, U14: SN74LVC2G17, Package_TO_SOT_SMD:SOT-363_SC-70-6, symbol myStuff:SN74LVC2G17
Connections:
- wire segments 88 -> 97
- no-connect marks 25 -> 23
Other:
- note added: "1 MHz clk input"
- note added: "Use PCNT and INT\nfor time-keeping\nhttps://github.com/espressif/esp-idf/blob/master/tools/unit-test-app/components/unity/ref_clock.c"
- note added: "WS2811 LED strip"
Changed lines of the file:
@@
 L power:GND #PWR0108
 U 1 1 5A1F3E37
-P 2650 3850
-F 0 "#PWR0108" H 2650 3600 50  0001 C CNN
-F 1 "GND" H 2500 3800 50  0000 C CNN
-F 2 "" H 2650 3850 50  0001 C CNN
-F 3 "" H 2650 3850 50  0001 C CNN
-	1    2650 3850
+P 3000 4750
+F 0 "#PWR0108" H 3000 4500 50  0001 C CNN
+F 1 "GND" H 2850 4700 50  0000 C CNN
+F 2 "" H 3000 4750 50  0001 C CNN
+F 3 "" H 3000 4750 50  0001 C CNN
+	1    3000 4750
 	1    0    0    -1
 $EndComp
@@
 L Device:C C1
 U 1 1 5A1F4174
-P 2650 3650
-F 0 "C1" V 2450 3700 50  0000 R CNN
-F 1 "1u" V 2450 3950 50  0000 R CNN
-F 2 "Capacitor_SMD:C_0805_2012Metric" H 2688 3500 50  0001 C CNN
-F 3 "" H 2650 3650 50  0001 C CNN
-F 4 "" H 100 -3200 50  0001 C CNN "DPN"
-	1    2650 3650
-	-1   0    0    1
-$EndComp
-Wire Wire Line
-	2650 3850 2650 3800
-Wire Wire Line
-	2650 3450 2650 3500
+P 3000 4550
+F 0 "C1" V 2800 4600 50  0000 R CNN
+F 1 "1u" V 2800 4850 50  0000 R CNN
+F 2 "Capacitor_SMD:C_0805_2012Metric" H 3038 4400 50  0001 C CNN
+F 3 "" H 3000 4550 50  0001 C CNN
+F 4 "" H 450 -2300 50  0001 C CNN "DPN"
+	1    3000 4550
+	-1   0    0    1
+$EndComp
+Wire Wire Line
+	3000 4750 3000 4700
+Wire Wire Line
+	3000 4350 3000 4400
 $Comp
 L power:GND #PWR0109
@@
 NoConn ~ 4050 1750
 NoConn ~ 4050 2250
-NoConn ~ 4050 2650
-NoConn ~ 4050 2750
 NoConn ~ 5400 3100
 NoConn ~ 4700 3100
@@
 	1    0    0    -1
 $EndComp
-$Comp
-L myStuff:74LVC3G34DP U1
-U 1 1 5B04A3F0
-P 2650 2800
-F 0 "U1" H 2650 2650 50  0000 C CNN
-F 1 "74LVC3G34DP" H 2200 2900 50  0000 C CNN
-F 2 "Package_SO:VSSOP-8_2.4x2.1mm_P0.5mm" H 2300 2400 50  0001 C CNN
-F 3 "http://www.nxp.com/documents/data_sheet/74LVC3G34.pdf" H 2550 2300 50  0001 C CNN
-F 4 "568-8987-1-ND" H 2750 3000 60  0001 C CNN "DPN"
-	1    2650 2800
-	-1   0    0    1
-$EndComp
-$Comp
-L myStuff:74LVC3G34DP U1
-U 2 1 5B04A4B8
-P 2650 2450
-F 0 "U1" H 2700 2350 50  0000 C CNN
-F 1 "74LVC3G34DP" H 2200 2550 50  0000 C CNN
-F 2 "Package_SO:VSSOP-8_2.4x2.1mm_P0.5mm" H 2300 2050 50  0001 C CNN
-F 3 "http://www.nxp.com/documents/data_sheet/74LVC3G34.pdf" H 2550 1950 50  0001 C CNN
-F 4 "568-8987-1-ND" H 2750 2650 60  0001 C CNN "DPN"
-	2    2650 2450
-	-1   0    0    1
-$EndComp
-$Comp
-L myStuff:74LVC3G34DP U1
-U 3 1 5B04A58F
-P 2650 2100
-F 0 "U1" H 2650 1950 50  0000 C CNN
-F 1 "74LVC3G34DP" H 2200 2200 50  0000 C CNN
-F 2 "Package_SO:VSSOP-8_2.4x2.1mm_P0.5mm" H 2300 1700 50  0001 C CNN
-F 3 "http://www.nxp.com/documents/data_sheet/74LVC3G34.pdf" H 2550 1600 50  0001 C CNN
-F 4 "568-8987-1-ND" H 2750 2300 60  0001 C CNN "DPN"
-	3    2650 2100
-	-1   0    0    1
-$EndComp
 Wire Wire Line
 	1950 2250 2050 2250
@@
 L power:VCC #PWR0136
 U 1 1 5B066227
-P 2650 3450
-F 0 "#PWR0136" H 2650 3300 50  0001 C CNN
-F 1 "VCC" H 2667 3623 50  0000 C CNN
-F 2 "" H 2650 3450 50  0001 C CNN
-F 3 "" H 2650 3450 50  0001 C CNN
-	1    2650 3450
-	1    0    0    -1
-$EndComp
+P 3000 4350
+F 0 "#PWR0136" H 3000 4200 50  0001 C CNN
+F 1 "VCC" H 3017 4523 50  0000 C CNN
+F 2 "" H 3000 4350 50  0001 C CNN
+F 3 "" H 3000 4350 50  0001 C CNN
+	1    3000 4350
+	1    0    0    -1
+$EndComp
+$Comp
+L myStuff:SN74LVC2G17 U1
+U 2 1 5B025765
+P 2650 2450
+F 0 "U1" H 2800 2550 50  0000 C CNN
+F 1 "SN74LVC2G17" H 2200 2550 50  0000 C CNN
+F 2 "Package_TO_SOT_SMD:SOT-363_SC-70-6" H 2650 2450 50  0001 C CNN
+F 3 "http://www.ti.com/lit/ds/symlink/sn74lvc2g17.pdf" H 2650 2201 50  0001 C CNN
+	2    2650 2450
+	-1   0    0    1
+$EndComp
+$Comp
+L myStuff:SN74LVC2G17 U1
+U 1 1 5B02595A
+P 2650 2800
+F 0 "U1" H 2800 2900 50  0000 C CNN
+F 1 "SN74LVC2G17" H 2200 2900 50  0000 C CNN
+F 2 "Package_TO_SOT_SMD:SOT-363_SC-70-6" H 2650 2800 50  0001 C CNN
+F 3 "http://www.ti.com/lit/ds/symlink/sn74lvc2g17.pdf" H 2650 2551 50  0001 C CNN
+	1    2650 2800
+	-1   0    0    1
+$EndComp
+$Comp
+L myStuff:SN74LVC2G17 U14
+U 1 1 5B025960
+P 2650 2100
+F 0 "U14" H 2800 2200 50  0000 C CNN
+F 1 "SN74LVC2G17" H 2200 2200 50  0000 C CNN
+F 2 "Package_TO_SOT_SMD:SOT-363_SC-70-6" H 2650 2100 50  0001 C CNN
+F 3 "http://www.ti.com/lit/ds/symlink/sn74lvc2g17.pdf" H 2650 1851 50  0001 C CNN
+	1    2650 2100
+	-1   0    0    1
+$EndComp
+$Comp
+L myStuff:SN74LVC2G17 U14
+U 2 1 5B0282F9
+P 2650 3250
+F 0 "U14" H 2800 3350 50  0000 C CNN
+F 1 "SN74LVC2G17" H 2200 3350 50  0000 C CNN
+F 2 "Package_TO_SOT_SMD:SOT-363_SC-70-6" H 2650 3250 50  0001 C CNN
+F 3 "http://www.ti.com/lit/ds/symlink/sn74lvc2g17.pdf" H 2650 3001 50  0001 C CNN
+	2    2650 3250
+	-1   0    0    1
+$EndComp
+Wire Wire Line
+	4050 2650 3750 2650
+Wire Wire Line
+	3750 2650 3750 3250
+Wire Wire Line
+	3750 3250 3100 3250
+$Comp
+L power:GND #PWR02
+U 1 1 5B03A1E0
+P 2050 3350
+F 0 "#PWR02" H 2050 3100 50  0001 C CNN
+F 1 "GND" V 2050 3150 50  0000 C CNN
+F 2 "" H 2050 3350 50  0001 C CNN
+F 3 "" H 2050 3350 50  0001 C CNN
+	1    2050 3350
+	0    -1   -1   0
+$EndComp
+Wire Wire Line
+	2200 3250 2050 3250
+$Comp
+L power:+5V #PWR01
+U 1 1 5B0446DD
+P 2050 3150
+F 0 "#PWR01" H 2050 3000 50  0001 C CNN
+F 1 "+5V" H 2065 3323 50  0000 C CNN
+F 2 "" H 2050 3150 50  0001 C CNN
+F 3 "" H 2050 3150 50  0001 C CNN
+	1    2050 3150
+	1    0    0    -1
+$EndComp
+Text Notes 1000 3200 0    50   ~ 0
+WS2811 LED strip
+$Comp
+L Connector_Generic:Conn_01x04 J7
+U 1 1 5B05FBD7
+P 1850 3250
+F 0 "J7" H 2000 3100 50  0000 C CNN
+F 1 "Conn_01x04" H 2150 3200 50  0000 C CNN
+F 2 "Connector_PinHeader_2.54mm:PinHeader_1x04_P2.54mm_Vertical" H 1850 3250 50  0001 C CNN
+F 3 "~" H 1850 3250 50  0001 C CNN
+	1    1850 3250
+	-1   0    0    -1
+$EndComp
+$Comp
+L power:GND #PWR04
+U 1 1 5B0310DE
+P 2500 4750
+F 0 "#PWR04" H 2500 4500 50  0001 C CNN
+F 1 "GND" H 2350 4700 50  0000 C CNN
+F 2 "" H 2500 4750 50  0001 C CNN
+F 3 "" H 2500 4750 50  0001 C CNN
+	1    2500 4750
+	1    0    0    -1
+$EndComp
+$Comp
+L Device:C C7
+U 1 1 5B0310E5
+P 2500 4550
+F 0 "C7" V 2300 4600 50  0000 R CNN
+F 1 "1u" V 2300 4850 50  0000 R CNN
+F 2 "Capacitor_SMD:C_0805_2012Metric" H 2538 4400 50  0001 C CNN
+F 3 "" H 2500 4550 50  0001 C CNN
+F 4 "" H -50 -2300 50  0001 C CNN "DPN"
+	1    2500 4550
+	-1   0    0    1
+$EndComp
+Wire Wire Line
+	2500 4750 2500 4700
+Wire Wire Line
+	2500 4350 2500 4400
+$Comp
+L power:VCC #PWR03
+U 1 1 5B0310ED
+P 2500 4350
+F 0 "#PWR03" H 2500 4200 50  0001 C CNN
+F 1 "VCC" H 2517 4523 50  0000 C CNN
+F 2 "" H 2500 4350 50  0001 C CNN
+F 3 "" H 2500 4350 50  0001 C CNN
+	1    2500 4350
+	1    0    0    -1
+$EndComp
+Wire Wire Line
+	4050 2750 3850 2750
+Wire Wire Line
+	3850 2750 3850 3450
+Wire Wire Line
+	3850 3450 2050 3450
+Text Notes 1000 3450 0    50   ~ 0
+1 MHz clk input
+Text Notes 950  3800 0    50   ~ 0
+Use PCNT and INT\nfor time-keeping\nhttps://github.com/espressif/esp-idf/blob/master/tools/unit-test-app/components/unity/ref_clock.c
 $EndSCHEMATC

Commit message: Decided for 12V input voltage
Parts:
- removed C3: 10u, Capacitor_SMD:C_1210_3225Metric, symbol Device:C
- removed C4, C7: 1u, Capacitor_SMD:C_0805_2012Metric, symbol Device:C
- removed U1, U14: SN74LVC2G17, Package_TO_SOT_SMD:SOT-363_SC-70-6, symbol myStuff:SN74LVC2G17
- removed U2: LM317EMP, SOT-223, symbol myStuff:LM317EMP
- added D1: B5819WS, Diode_SMD:D_SOD-323, symbol Device:D_Schottky
- added Q1, Q2, Q3: BSS138, Package_TO_SOT_SMD:SOT-23, symbol myStuff:BSS138_ok
- added R14, R15, R16, R17: 10k, Resistor_SMD:R_0805_2012Metric, symbol Device:R
- added R18: 50R, Resistor_SMD:R_0805_2012Metric, symbol Device:R
- added U1: DCDC_mod, myStuff:ebay_dcdc, symbol myStuff:DCDC_mod
- C1: value 1u -> 10u; footprint Capacitor_SMD:C_0805_2012Metric -> Capacitor_SMD:C_1210_3225Metric
- R2: value 590R -> 10k
- R3: value 1k -> 10k
Connections:
- net labels added: +12V
- net labels removed: +5V, VCC
- wire segments 97 -> 83
Other:
- note removed: "3.419 V"
