File: pcb/nixie/tubes.sch (KiCad schematic (older format))
At the start: 24 parts, among them U10 nixie_8422, U11 nixie_8422, U12 nixie_8422, U5 nixie_8422, U6 HV5530, U7 HV5530, U8 nixie_8422, U9 nixie_8422

Commit message: pff
Parts:
- added J1, J3, J4, J5: Conn_01x32, Connector_PinHeader_1.27mm:PinHeader_1x32_P1.27mm_Vertical, symbol Connector_Generic:Conn_01x32
- NE1, NE2, NE3, NE4: footprint Valve:Valve_Glimm -> Connector_PinHeader_2.54mm:PinHeader_1x02_P2.54mm_Vertical
Connections:
- wire segments 194 -> 260

Commit message: Not sure where im going here
Parts:
- J1, J4: footprint Connector_PinHeader_1.27mm:PinHeader_1x32_P1.27mm_Vertical -> Connector_PinHeader_2.54mm:PinHeader_2x16_P2.54mm_Horizontal
- J3, J5: footprint Connector_PinHeader_1.27mm:PinHeader_1x32_P1.27mm_Vertical -> Connector_PinHeader_2.54mm:PinHeader_2x16_P2.54mm_Vertical
Connections:
- wire segments 260 -> 256

Commit message: PCB work
Parts:
- J1, J4: footprint Connector_PinHeader_2.54mm:PinHeader_2x16_P2.54mm_Horizontal -> Connector_PinHeader_2.54mm:PinHeader_1x32_P2.54mm_Vertical
- J3, J5: footprint Connector_PinHeader_2.54mm:PinHeader_2x16_P2.54mm_Vertical -> Connector_PinHeader_2.54mm:PinHeader_1x32_P2.54mm_Vertical
Connections:
- wire segments 256 -> 258

Commit message: Added MCP1630 idea
Parts:
- renumbered C7 to C?, C8 to C?, J1 to J?, J3 to J?, J4 to J?, J5 to J?, NE3 to NE?, NE4 to NE?, NE1 to NE?, NE2 to NE?, R8 to R?, R7 to R?, R11 to R?, R12 to R?, R15 to R?, R16 to R?, R13 to R?, R14 to R?, R9 to R?, R10 to R?, U5 to U?, U8 to U?, U9 to U?, U10 to U?, U11 to U?, U12 to U?, U6 to U?, U7 to U?

Commit message: tricky
Parts:
- gave numbers to parts that had none: 28
Connections:
- net labels added: +5V
- net labels removed: +12V

Commit message: Decided for 12V input voltage
Connections:
- net labels added: +12V
- net labels removed: +5V
Changed lines of the file:
@@
 	6000 5850 6250 5850
 $Comp
-L power:+5V #PWR0134
-U 1 1 5B03FE18
+L power:+12V #PWR0139
+U 1 1 5B17D9CB
 P 1450 4000
-F 0 "#PWR0134" H 1450 3850 50  0001 C CNN
-F 1 "+5V" H 1465 4173 50  0000 C CNN
+F 0 "#PWR0139" H 1450 3850 50  0001 C CNN
+F 1 "+12V" H 1465 4173 50  0000 C CNN
 F 2 "" H 1450 4000 50  0001 C CNN
 F 3 "" H 1450 4000 50  0001 C CNN
@@
 $EndComp
 $Comp
-L power:+5V #PWR0135
-U 1 1 5B03FFC2
+L power:+12V #PWR0140
+U 1 1 5B17DA25
 P 1400 5850
-F 0 "#PWR0135" H 1400 5700 50  0001 C CNN
-F 1 "+5V" H 1415 6023 50  0000 C CNN
+F 0 "#PWR0140" H 1400 5700 50  0001 C CNN
+F 1 "+12V" H 1415 6023 50  0000 C CNN
 F 2 "" H 1400 5850 50  0001 C CNN
 F 3 "" H 1400 5850 50  0001 C CNN
