File: pcb/nixie/nixie.kicad_pcb (KiCad board)
At the start: 2 copper layers, 144 x 117 mm, 45 parts, among them J2 Conn_01x02, P1 TTL_232R_3V3, Q1 Q_NMOS_DGS, U1 LM317EMP, U10 nixie_8422, U11 nixie_8422, U12 nixie_8422, U2 ESP-WROOM-32, U3 TACTILE, U4 TACTILE, U5 nixie_8422, U6 HV5530, U7 HV5530, U8 nixie_8422, U9 nixie_8422

Commit message: pff
Parts:
- added J1: Conn_01x32, Connector_PinHeader_1.27mm:PinHeader_1x32_P1.27mm_Vertical, F.Cu at (39.5, 144.5)
- added J3: Conn_01x32, Connector_PinHeader_1.27mm:PinHeader_1x32_P1.27mm_Vertical, F.Cu at (114.0, 144.5)
- added J4: Conn_01x32, Connector_PinHeader_1.27mm:PinHeader_1x32_P1.27mm_Vertical, F.Cu at (39.5, 132.0)
- added J5: Conn_01x32, Connector_PinHeader_1.27mm:PinHeader_1x32_P1.27mm_Vertical, F.Cu at (114.0, 132.0)
- NE1, NE2, NE3, NE4: footprint Valve:Valve_Glimm -> Connector_PinHeader_2.54mm:PinHeader_1x02_P2.54mm_Vertical
- moved U7 10.3 mm to (133.0, 115.5), turned to 180 degrees
- moved U6 7.02 mm to (54.5, 116.0)
- moved U11 4.53 mm to (137.5, 160.5)
- moved U12 4.53 mm to (158.5, 160.5)
- moved U5 4.53 mm to (37.5, 160.5)
- moved U8 4.53 mm to (58.5, 160.5)
- moved NE1 3.54 mm to (73.0, 167.5), turned to 180 degrees
- moved NE2 3.54 mm to (73.0, 156.0), turned to 180 degrees
- moved NE3 3.20 mm to (123.0, 156.0), turned to 180 degrees
- moved NE4 3.20 mm to (123.0, 167.5), turned to 180 degrees
- moved U10 0.50 mm to (108.5, 160.5)
- moved U9 0.50 mm to (87.5, 160.5)

Commit message: Not sure where im going here
Parts:
- J1, J4: footprint Connector_PinHeader_1.27mm:PinHeader_1x32_P1.27mm_Vertical -> Connector_PinHeader_2.54mm:PinHeader_2x16_P2.54mm_Horizontal; moved to B.Cu
- J3, J5: footprint Connector_PinHeader_1.27mm:PinHeader_1x32_P1.27mm_Vertical -> Connector_PinHeader_2.54mm:PinHeader_2x16_P2.54mm_Vertical
- R10, R11, R12, R13, R14, R15, R16, R7, R8, R9, U6: moved to B.Cu
- moved R9 149.8 mm to (73.1, 171.9), turned to 90 degrees
- moved R7 134.0 mm to (42.1, 145.3), turned to 90 degrees
- moved R8 126.1 mm to (62.4, 145.3), turned to 270 degrees
- moved R10 107.6 mm to (73.1, 160.2), turned to 90 degrees
- moved R13 104.8 mm to (123.4, 160.5)
- moved R14 98.8 mm to (118.3, 163.0)
- moved R16 94.4 mm to (161.5, 145.3), turned to 270 degrees
- moved R12 89.5 mm to (113.2, 145.3), turned to 270 degrees
- moved R15 88.5 mm to (141.2, 145.3), turned to 270 degrees
- moved J4 85.6 mm to (114.5, 173.2), turned to 270 degrees
- moved R11 75.8 mm to (91.4, 145.3), turned to 270 degrees
- moved J3 71.6 mm to (43.4, 132.6)
- moved J1 28.8 mm to (42.1, 173.2), turned to 270 degrees
- moved U6 6.64 mm to (59.9, 119.9)
- moved J5 0.76 mm to (114.5, 132.6)
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Connections:
- J1 pad 32: HT -> Net-(J1-Pad32)
- J3 pad 1: /tubes/n2_0 -> /tubes/n5_0
- J3 pad 10: /tubes/n2_9 -> /tubes/n5_9
- J3 pad 11: /tubes/colons_0 -> /tubes/n4_0
- J3 pad 12: /tubes/n1_0 -> /tubes/n4_1
- J3 pad 13: /tubes/n1_1 -> /tubes/n4_2
- J3 pad 14: /tubes/n1_2 -> /tubes/n4_3
- J3 pad 15: /tubes/n1_3 -> /tubes/n4_4
- J3 pad 16: /tubes/n1_4 -> /tubes/n4_5
- J3 pad 17: /tubes/n1_5 -> /tubes/n4_6
- J3 pad 18: /tubes/n1_6 -> /tubes/n4_7
- J3 pad 19: /tubes/n1_7 -> /tubes/n4_8
- J3 pad 2: /tubes/n2_1 -> /tubes/n5_1
- J3 pad 20: /tubes/n1_8 -> /tubes/n4_9
- J3 pad 21: /tubes/n1_9 -> /tubes/colons_1
- J3 pad 22: /tubes/n0_0 -> /tubes/n3_0
- J3 pad 23: /tubes/n0_1 -> /tubes/n3_1
- J3 pad 24: /tubes/n0_2 -> /tubes/n3_2
- J3 pad 25: /tubes/n0_3 -> /tubes/n3_3
- J3 pad 26: /tubes/n0_4 -> /tubes/n3_4
- J3 pad 27: /tubes/n0_5 -> /tubes/n3_5
- J3 pad 28: /tubes/n0_6 -> /tubes/n3_6
- J3 pad 29: /tubes/n0_7 -> /tubes/n3_7
- J3 pad 3: /tubes/n2_2 -> /tubes/n5_2
- J3 pad 30: /tubes/n0_8 -> /tubes/n3_8
- J3 pad 31: /tubes/n0_9 -> /tubes/n3_9
- J3 pad 32: HT -> Net-(J3-Pad32)
- J3 pad 4: /tubes/n2_3 -> /tubes/n5_3
- J3 pad 5: /tubes/n2_4 -> /tubes/n5_4
- J3 pad 6: /tubes/n2_5 -> /tubes/n5_5
- J3 pad 7: /tubes/n2_6 -> /tubes/n5_6
- J3 pad 8: /tubes/n2_7 -> /tubes/n5_7
- J3 pad 9: /tubes/n2_8 -> /tubes/n5_8
- J4 pad 1: /tubes/n5_0 -> /tubes/n2_0
- J4 pad 10: /tubes/n5_9 -> /tubes/n2_9
- J4 pad 11: /tubes/n4_0 -> /tubes/colons_0
- J4 pad 12: /tubes/n4_1 -> /tubes/n1_0
- J4 pad 13: /tubes/n4_2 -> /tubes/n1_1
- J4 pad 14: /tubes/n4_3 -> /tubes/n1_2
- J4 pad 15: /tubes/n4_4 -> /tubes/n1_3
- J4 pad 16: /tubes/n4_5 -> /tubes/n1_4
- J4 pad 17: /tubes/n4_6 -> /tubes/n1_5
- J4 pad 18: /tubes/n4_7 -> /tubes/n1_6
- J4 pad 19: /tubes/n4_8 -> /tubes/n1_7
- J4 pad 2: /tubes/n5_1 -> /tubes/n2_1
- J4 pad 20: /tubes/n4_9 -> /tubes/n1_8
- J4 pad 21: /tubes/colons_1 -> /tubes/n1_9
- J4 pad 22: /tubes/n3_0 -> /tubes/n0_0
- J4 pad 23: /tubes/n3_1 -> /tubes/n0_1
- J4 pad 24: /tubes/n3_2 -> /tubes/n0_2
- J4 pad 25: /tubes/n3_3 -> /tubes/n0_3
- J4 pad 26: /tubes/n3_4 -> /tubes/n0_4
- J4 pad 27: /tubes/n3_5 -> /tubes/n0_5
- J4 pad 28: /tubes/n3_6 -> /tubes/n0_6
- J4 pad 29: /tubes/n3_7 -> /tubes/n0_7
- J4 pad 3: /tubes/n5_2 -> /tubes/n2_2
- J4 pad 30: /tubes/n3_8 -> /tubes/n0_8
- J4 pad 31: /tubes/n3_9 -> /tubes/n0_9
- J4 pad 32: HT -> Net-(J4-Pad32)
- J4 pad 4: /tubes/n5_3 -> /tubes/n2_3
- J4 pad 5: /tubes/n5_4 -> /tubes/n2_4
- J4 pad 6: /tubes/n5_5 -> /tubes/n2_5
- J4 pad 7: /tubes/n5_6 -> /tubes/n2_6
- J4 pad 8: /tubes/n5_7 -> /tubes/n2_7
- J4 pad 9: /tubes/n5_8 -> /tubes/n2_8
- J5 pad 32: HT -> Net-(J5-Pad32)
Routing:
- net /tubes/n4_7: track 0.00 -> 24.8 mm
- net /tubes/n4_9: track 0.00 -> 22.3 mm
- net /tubes/n3_0: track 0.00 -> 19.5 mm
- net /tubes/n3_2: track 0.00 -> 16.1 mm
- net /tubes/n3_4: track 0.00 -> 14.7 mm
- net /tubes/n3_6: track 0.00 -> 12.1 mm
- net /tubes/n3_8: track 0.00 -> 9.33 mm
- net Net-(J1-Pad32): track 0.00 -> 5.97 mm
Other:
- net class Default: clearance 0.2 -> 0.3; trace_width 0.25 -> 0.3; via_dia 0.8 -> 1.2; via_drill 0.4 -> 0.6
- rule trace_clearance: 0.2 -> 0.3
- rule trace_min: 0.2 -> 0.3
- rule via_min_drill: 0.3 -> 0.6
- rule via_min_size: 0.4 -> 1.2

Commit message: PCB work
Parts:
- added C9: 10u, Capacitor_SMD:C_2010_5025Metric, F.Cu at (102.6, 123.7)
- added Q2: 2N7002, Package_TO_SOT_SMD:SOT-23, B.Cu at (79.3, 103.3)
- added Q3: 2N7002, Package_TO_SOT_SMD:SOT-23, B.Cu at (82.1, 106.2)
- added Q4: 2N7002, Package_TO_SOT_SMD:SOT-23, B.Cu at (69.2, 103.5)
- added R17: 1k, Resistor_SMD:R_0805_2012Metric, B.Cu at (77.1, 101.0)
- added R18: 1k, Resistor_SMD:R_0805_2012Metric, B.Cu at (84.5, 108.5)
- added R19: 1k, Resistor_SMD:R_0805_2012Metric, B.Cu at (71.5, 101.3)
- added REF**: MountingHole_3.2mm_M3, MountingHole:MountingHole_3.2mm_M3, F.Cu at (167.0, 99.0)
- added REF**: MountingHole_3.2mm_M3, MountingHole:MountingHole_3.2mm_M3, F.Cu at (29.0, 132.0)
- added REF**: MountingHole_3.2mm_M3, MountingHole:MountingHole_3.2mm_M3, F.Cu at (167.0, 132.0)
- added REF**: MountingHole_3.2mm_M3, MountingHole:MountingHole_3.2mm_M3, F.Cu at (29.0, 99.0)
- added REF**: MountingHole_3.2mm_M3, MountingHole:MountingHole_3.2mm_M3, F.Cu at (29.0, 55.0)
- added REF**: MountingHole_3.2mm_M3, MountingHole:MountingHole_3.2mm_M3, F.Cu at (29.0, 22.0)
- added REF**: MountingHole_3.2mm_M3, MountingHole:MountingHole_3.2mm_M3, F.Cu at (167.0, 55.0)
- added REF**: MountingHole_3.2mm_M3, MountingHole:MountingHole_3.2mm_M3, F.Cu at (167.0, 22.0)
- C1, C2, C3, C4, C6, C7, C8, P1, R1, R2, R3, R4, R5, R6, U3, U4, U7: moved to B.Cu
- J1, J4: footprint Connector_PinHeader_2.54mm:PinHeader_2x16_P2.54mm_Horizontal -> Connector_PinHeader_2.54mm:PinHeader_1x32_P2.54mm_Vertical
- J3, J5: footprint Connector_PinHeader_2.54mm:PinHeader_2x16_P2.54mm_Vertical -> Connector_PinHeader_2.54mm:PinHeader_1x32_P2.54mm_Vertical
- moved J4 155.6 mm to (82.0, 21.0)
- moved R9 148.4 mm to (64.1, 23.8), turned to 270 degrees
- moved R10 136.5 mm to (69.2, 23.8), turned to 270 degrees
- moved NE1 125.3 mm to (73.0, 42.2), turned to 0 degrees
- moved NE4 125.3 mm to (123.0, 42.2), turned to 0 degrees
- moved NE2 123.8 mm to (73.0, 32.2), turned to 0 degrees
- moved NE3 123.8 mm to (123.0, 32.2), turned to 0 degrees
- moved R11 122.7 mm to (74.3, 23.8)
- moved R7 122.3 mm to (56.5, 23.8)
- moved U10 122.0 mm to (108.5, 38.5)
- moved U11 122.0 mm to (137.5, 38.5)
- moved U12 122.0 mm to (158.5, 38.5)
- moved U5 122.0 mm to (37.5, 38.5)
- moved U8 122.0 mm to (58.5, 38.5)
- moved U9 122.0 mm to (87.5, 38.5)
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Connections:
- J1 pad 1: /tubes/n5_0 -> GND
- J1 pad 11: /tubes/n4_0 -> /tubes/n5_0
- J1 pad 21: /tubes/colons_1 -> /tubes/n4_0
- J1 pad 22: /tubes/n3_0 -> /tubes/colons_1
- J1 pad 32: Net-(J1-Pad32) -> /tubes/n3_0
- J3 pad 1: /tubes/n5_0 -> GND
- J3 pad 11: /tubes/n4_0 -> /tubes/n5_0
- J3 pad 21: /tubes/colons_1 -> /tubes/n4_0
- J3 pad 22: /tubes/n3_0 -> /tubes/colons_1
- J3 pad 32: Net-(J3-Pad32) -> /tubes/n3_0
- J4 pad 1: /tubes/n2_0 -> HT
- J4 pad 10: /tubes/n2_9 -> /tubes/n2_8
- J4 pad 11: /tubes/colons_0 -> /tubes/n2_7
- J4 pad 12: /tubes/n1_0 -> /tubes/colons_0
- J4 pad 13: /tubes/n1_1 -> /tubes/n1_6
- J4 pad 14: /tubes/n1_2 -> /tubes/n1_5
- J4 pad 15: /tubes/n1_3 -> /tubes/n1_4
- J4 pad 16: /tubes/n1_4 -> /tubes/n1_3
- J4 pad 17: /tubes/n1_5 -> /tubes/n1_2
- J4 pad 18: /tubes/n1_6 -> /tubes/n1_1
- J4 pad 19: /tubes/n1_7 -> /tubes/n1_0
- J4 pad 2: /tubes/n2_1 -> /tubes/n2_6
- J4 pad 20: /tubes/n1_8 -> /tubes/n1_9
- J4 pad 21: /tubes/n1_9 -> /tubes/n1_8
- J4 pad 22: /tubes/n0_0 -> /tubes/n1_7
- J4 pad 23: /tubes/n0_1 -> /tubes/n0_6
- J4 pad 24: /tubes/n0_2 -> /tubes/n0_5
- J4 pad 25: /tubes/n0_3 -> /tubes/n0_4
- J4 pad 26: /tubes/n0_4 -> /tubes/n0_3
- J4 pad 27: /tubes/n0_5 -> /tubes/n0_2
- J4 pad 28: /tubes/n0_6 -> /tubes/n0_1
- J4 pad 29: /tubes/n0_7 -> /tubes/n0_0
- J4 pad 3: /tubes/n2_2 -> /tubes/n2_5
- J4 pad 30: /tubes/n0_8 -> /tubes/n0_9
- J4 pad 31: /tubes/n0_9 -> /tubes/n0_8
- J4 pad 32: Net-(J4-Pad32) -> /tubes/n0_7
- J4 pad 4: /tubes/n2_3 -> /tubes/n2_4
- J4 pad 5: /tubes/n2_4 -> /tubes/n2_3
- J4 pad 6: /tubes/n2_5 -> /tubes/n2_2
- J4 pad 7: /tubes/n2_6 -> /tubes/n2_1
- J4 pad 8: /tubes/n2_7 -> /tubes/n2_0
- J4 pad 9: /tubes/n2_8 -> /tubes/n2_9
- J5 pad 1: /tubes/n2_0 -> HT
- J5 pad 10: /tubes/n2_9 -> /tubes/n2_8
- J5 pad 11: /tubes/colons_0 -> /tubes/n2_7
- J5 pad 12: /tubes/n1_0 -> /tubes/colons_0
- J5 pad 13: /tubes/n1_1 -> /tubes/n1_6
- J5 pad 14: /tubes/n1_2 -> /tubes/n1_5
- J5 pad 15: /tubes/n1_3 -> /tubes/n1_4
- J5 pad 16: /tubes/n1_4 -> /tubes/n1_3
- J5 pad 17: /tubes/n1_5 -> /tubes/n1_2
- J5 pad 18: /tubes/n1_6 -> /tubes/n1_1
- J5 pad 19: /tubes/n1_7 -> /tubes/n1_0
- J5 pad 2: /tubes/n2_1 -> /tubes/n2_6
- J5 pad 20: /tubes/n1_8 -> /tubes/n1_9
- J5 pad 21: /tubes/n1_9 -> /tubes/n1_8
- J5 pad 22: /tubes/n0_0 -> /tubes/n1_7
- J5 pad 23: /tubes/n0_1 -> /tubes/n0_6
- J5 pad 24: /tubes/n0_2 -> /tubes/n0_5
- J5 pad 25: /tubes/n0_3 -> /tubes/n0_4
- J5 pad 26: /tubes/n0_4 -> /tubes/n0_3
- J5 pad 27: /tubes/n0_5 -> /tubes/n0_2
- J5 pad 28: /tubes/n0_6 -> /tubes/n0_1
- J5 pad 29: /tubes/n0_7 -> /tubes/n0_0
- J5 pad 3: /tubes/n2_2 -> /tubes/n2_5
- J5 pad 30: /tubes/n0_8 -> /tubes/n0_9
- J5 pad 31: /tubes/n0_9 -> /tubes/n0_8
- J5 pad 32: Net-(J5-Pad32) -> /tubes/n0_7
- J5 pad 4: /tubes/n2_3 -> /tubes/n2_4
- J5 pad 5: /tubes/n2_4 -> /tubes/n2_3
- J5 pad 6: /tubes/n2_5 -> /tubes/n2_2
- J5 pad 7: /tubes/n2_6 -> /tubes/n2_1
- J5 pad 8: /tubes/n2_7 -> /tubes/n2_0
- J5 pad 9: /tubes/n2_8 -> /tubes/n2_9
- U2 pad 10: /tubes/clk -> Net-(Q4-Pad1)
- U2 pad 11: /tubes/dat -> Net-(Q3-Pad1)
- U2 pad 12: /tubes/nLatch -> Net-(Q2-Pad1)
- U6 pad 1: /tubes/n4_0 -> /tubes/colons_1
- U6 pad 10: /tubes/n4_9 -> /tubes/n4_2
- U6 pad 11: /tubes/colons_1 -> /tubes/n4_1
- U6 pad 12: /tubes/n3_0 -> /tubes/n5_0
- U6 pad 13: /tubes/n3_1 -> /tubes/n5_9
- U6 pad 14: /tubes/n3_2 -> /tubes/n5_8
- U6 pad 15: /tubes/n3_3 -> /tubes/n5_7
- U6 pad 16: /tubes/n3_4 -> /tubes/n5_6
- U6 pad 17: /tubes/n3_5 -> /tubes/n5_5
- U6 pad 18: /tubes/n3_6 -> /tubes/n5_4
- U6 pad 19: /tubes/n3_7 -> /tubes/n5_3
- U6 pad 2: /tubes/n4_1 -> /tubes/n4_0
- U6 pad 20: /tubes/n3_8 -> /tubes/n5_2
- U6 pad 21: /tubes/n3_9 -> /tubes/n5_1
- U6 pad 3: /tubes/n4_2 -> /tubes/n4_9
- U6 pad 35: /tubes/n5_0 -> /tubes/n3_0
- U6 pad 36: /tubes/n5_1 -> /tubes/n3_9
- U6 pad 37: /tubes/n5_2 -> /tubes/n3_8
- U6 pad 38: /tubes/n5_3 -> /tubes/n3_7
- U6 pad 39: /tubes/n5_4 -> /tubes/n3_6
- U6 pad 4: /tubes/n4_3 -> /tubes/n4_8
- U6 pad 40: /tubes/n5_5 -> /tubes/n3_5
- U6 pad 41: /tubes/n5_6 -> /tubes/n3_4
- U6 pad 42: /tubes/n5_7 -> /tubes/n3_3
- U6 pad 43: /tubes/n5_8 -> /tubes/n3_2
- U6 pad 44: /tubes/n5_9 -> /tubes/n3_1
- U6 pad 5: /tubes/n4_4 -> /tubes/n4_7
- U6 pad 6: /tubes/n4_5 -> /tubes/n4_6
- U6 pad 7: /tubes/n4_6 -> /tubes/n4_5
- U6 pad 8: /tubes/n4_7 -> /tubes/n4_4
- U6 pad 9: /tubes/n4_8 -> /tubes/n4_3
- U7 pad 1: /tubes/colons_0 -> /tubes/n2_7
- U7 pad 10: /tubes/n1_8 -> /tubes/n1_9
- U7 pad 11: /tubes/n1_9 -> /tubes/n1_8
- U7 pad 12: /tubes/n0_0 -> /tubes/n1_7
- U7 pad 13: /tubes/n0_1 -> /tubes/n0_6
- U7 pad 14: /tubes/n0_2 -> /tubes/n0_5
- U7 pad 15: /tubes/n0_3 -> /tubes/n0_4
- U7 pad 16: /tubes/n0_4 -> /tubes/n0_3
- U7 pad 17: /tubes/n0_5 -> /tubes/n0_2
- U7 pad 18: /tubes/n0_6 -> /tubes/n0_1
- U7 pad 19: /tubes/n0_7 -> /tubes/n0_0
- U7 pad 2: /tubes/n1_0 -> /tubes/colons_0
- U7 pad 20: /tubes/n0_8 -> /tubes/n0_9
- U7 pad 21: /tubes/n0_9 -> /tubes/n0_8
- U7 pad 22: Net-(U7-Pad22) -> /tubes/n0_7
- U7 pad 3: /tubes/n1_1 -> /tubes/n1_6
- U7 pad 35: /tubes/n2_0 -> Net-(U7-Pad35)
- U7 pad 36: /tubes/n2_1 -> /tubes/n2_6
- U7 pad 37: /tubes/n2_2 -> /tubes/n2_5
- U7 pad 38: /tubes/n2_3 -> /tubes/n2_4
- U7 pad 39: /tubes/n2_4 -> /tubes/n2_3
- U7 pad 4: /tubes/n1_2 -> /tubes/n1_5
- U7 pad 40: /tubes/n2_5 -> /tubes/n2_2
- U7 pad 41: /tubes/n2_6 -> /tubes/n2_1
- U7 pad 42: /tubes/n2_7 -> /tubes/n2_0
- U7 pad 43: /tubes/n2_8 -> /tubes/n2_9
- U7 pad 44: /tubes/n2_9 -> /tubes/n2_8
- U7 pad 5: /tubes/n1_3 -> /tubes/n1_4
- U7 pad 6: /tubes/n1_4 -> /tubes/n1_3
- U7 pad 7: /tubes/n1_5 -> /tubes/n1_2
- U7 pad 8: /tubes/n1_6 -> /tubes/n1_1
- U7 pad 9: /tubes/n1_7 -> /tubes/n1_0
Routing:
- net HT: track 0.00 -> 125.1 mm, vias 0 -> 2
- net /tubes/n2_6: track 0.00 -> 80.5 mm
- net /tubes/n0_7: track 0.00 -> 74.2 mm
- net /tubes/n5_1: track 0.00 -> 70.1 mm
- net /tubes/n2_5: track 0.00 -> 70.0 mm
- net /tubes/n0_8: track 0.00 -> 64.9 mm
- net /tubes/n3_9: track 0.00 -> 64.7 mm
- net /tubes/n2_4: track 0.00 -> 62.5 mm
- net /tubes/n5_2: track 0.00 -> 62.3 mm
- net /tubes/n0_9: track 0.00 -> 57.7 mm
- net /tubes/n0_6: track 0.00 -> 55.9 mm
- net /tubes/n5_3: track 0.00 -> 55.7 mm
- net /tubes/n3_0: track 19.5 -> 74.9 mm
- net /tubes/n1_6: track 0.00 -> 53.6 mm
- net /tubes/n0_0: track 0.00 -> 50.9 mm
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- added copper zone on B.Cu, net GND
- added copper zone on F.Cu, net GND
Other:
- board size 144 x 117 mm -> 144 x 116 mm

Commit message: tricky
Parts:
- removed C7, C8: 1u, Capacitor_SMD:C_0805_2012Metric
- removed C9: 10u, Capacitor_SMD:C_2010_5025Metric
- removed D1: D, Diode_SMD:D_1206_3216Metric
- removed L1: L, myStuff:cc_5022
- removed Q1: Q_NMOS_DGS, Package_TO_SOT_SMD:SOT-23
- removed Q2, Q3, Q4: 2N7002, Package_TO_SOT_SMD:SOT-23
- removed R14, R15, R16: 10k, Resistor_SMD:R_0805_2012Metric
- removed R17, R18, R19: 1k, Resistor_SMD:R_0805_2012Metric
- added J1: Conn_01x02, Connector_PinHeader_2.54mm:PinHeader_1x02_P2.54mm_Vertical, F.Cu at (127.6, 153.9)
- added U2: LM317EMP, SOT-223, F.Cu at (57.8, 102.1)
- C1: value 470n -> 1u; moved to F.Cu
- C3: footprint Capacitor_SMD:C_2010_5025Metric -> Capacitor_SMD:C_1210_3225Metric
- C5: value 10u -> 1u; footprint Capacitor_SMD:C_2010_5025Metric -> Capacitor_SMD:C_0805_2012Metric
- C6: value 100n -> 1u
- R2: value 10R -> 590R
- R3: value 590R -> 1k
- R4: value 1k -> 10k
- R5: value 1M3 -> 10k
- R6: value 7k15 -> 10k
- U1: value LM317EMP -> 74LVC3G34DP; footprint SOT-223 -> Package_SO:VSSOP-8_2.4x2.1mm_P0.5mm; moved to B.Cu
- moved C2 71.7 mm to (28.4, 124.2)
- moved R1 70.3 mm to (32.1, 124.2)
- moved C4 36.3 mm to (58.6, 103.0)
- moved C1 34.2 mm to (73.6, 102.3), turned to 270 degrees
- moved C3 31.5 mm to (51.5, 103.7), turned to 270 degrees
- moved U1 21.4 mm to (73.8, 102.1), turned to 0 degrees
- renumbered J1 to J6, U9 to U10, U10 to U11, U11 to U12, U12 to U13, U2 to U3, U3 to U4, U4 to U5, U5 to U6, U6 to U7, U7 to U8, U8 to U9
Connections:
- C1 pad 2: +3V3 -> +5V
- C2 pad 2: +12V -> +3V3
- C3 pad 1: +12V -> +5V
- C5 pad 1: HT -> +5V
- C6 pad 1: /vHtMon -> +5V
- J2 pad 2: +12V -> HT
- J4 pad 1: HT -> GND
- J4 pad 10: /tubes/n2_8 -> /tubes/n5_9
- J4 pad 11: /tubes/n2_7 -> /tubes/n5_0
- J4 pad 12: /tubes/colons_0 -> /tubes/n4_1
- J4 pad 13: /tubes/n1_6 -> /tubes/n4_2
- J4 pad 14: /tubes/n1_5 -> /tubes/n4_3
- J4 pad 15: /tubes/n1_4 -> /tubes/n4_4
- J4 pad 16: /tubes/n1_3 -> /tubes/n4_5
- J4 pad 17: /tubes/n1_2 -> /tubes/n4_6
- J4 pad 18: /tubes/n1_1 -> /tubes/n4_7
- J4 pad 19: /tubes/n1_0 -> /tubes/n4_8
- J4 pad 2: /tubes/n2_6 -> /tubes/n5_1
- J4 pad 20: /tubes/n1_9 -> /tubes/n4_9
- J4 pad 21: /tubes/n1_8 -> /tubes/n4_0
- J4 pad 22: /tubes/n1_7 -> /tubes/colons_1
- J4 pad 23: /tubes/n0_6 -> /tubes/n3_1
- J4 pad 24: /tubes/n0_5 -> /tubes/n3_2
- J4 pad 25: /tubes/n0_4 -> /tubes/n3_3
- J4 pad 26: /tubes/n0_3 -> /tubes/n3_4
- J4 pad 27: /tubes/n0_2 -> /tubes/n3_5
- J4 pad 28: /tubes/n0_1 -> /tubes/n3_6
- J4 pad 29: /tubes/n0_0 -> /tubes/n3_7
- J4 pad 3: /tubes/n2_5 -> /tubes/n5_2
- J4 pad 30: /tubes/n0_9 -> /tubes/n3_8
- J4 pad 31: /tubes/n0_8 -> /tubes/n3_9
- J4 pad 32: /tubes/n0_7 -> /tubes/n3_0
- J4 pad 4: /tubes/n2_4 -> /tubes/n5_3
- J4 pad 5: /tubes/n2_3 -> /tubes/n5_4
- J4 pad 6: /tubes/n2_2 -> /tubes/n5_5
- J4 pad 7: /tubes/n2_1 -> /tubes/n5_6
- J4 pad 8: /tubes/n2_0 -> /tubes/n5_7
- J4 pad 9: /tubes/n2_9 -> /tubes/n5_8
- J6 pad 1: GND -> HT
- J6 pad 10: /tubes/n5_9 -> /tubes/n2_8
- J6 pad 11: /tubes/n5_0 -> /tubes/n2_7
- J6 pad 12: /tubes/n4_1 -> /tubes/colons_0
- J6 pad 13: /tubes/n4_2 -> /tubes/n1_6
- J6 pad 14: /tubes/n4_3 -> /tubes/n1_5
- J6 pad 15: /tubes/n4_4 -> /tubes/n1_4
- J6 pad 16: /tubes/n4_5 -> /tubes/n1_3
- J6 pad 17: /tubes/n4_6 -> /tubes/n1_2
- J6 pad 18: /tubes/n4_7 -> /tubes/n1_1
- J6 pad 19: /tubes/n4_8 -> /tubes/n1_0
- J6 pad 2: /tubes/n5_1 -> /tubes/n2_6
- J6 pad 20: /tubes/n4_9 -> /tubes/n1_9
- J6 pad 21: /tubes/n4_0 -> /tubes/n1_8
- J6 pad 22: /tubes/colons_1 -> /tubes/n1_7
- J6 pad 23: /tubes/n3_1 -> /tubes/n0_6
- J6 pad 24: /tubes/n3_2 -> /tubes/n0_5
- J6 pad 25: /tubes/n3_3 -> /tubes/n0_4
- J6 pad 26: /tubes/n3_4 -> /tubes/n0_3
- J6 pad 27: /tubes/n3_5 -> /tubes/n0_2
- J6 pad 28: /tubes/n3_6 -> /tubes/n0_1
- J6 pad 29: /tubes/n3_7 -> /tubes/n0_0
- J6 pad 3: /tubes/n5_2 -> /tubes/n2_5
- J6 pad 30: /tubes/n3_8 -> /tubes/n0_9
- J6 pad 31: /tubes/n3_9 -> /tubes/n0_8
- J6 pad 32: /tubes/n3_0 -> /tubes/n0_7
- J6 pad 4: /tubes/n5_3 -> /tubes/n2_4
- J6 pad 5: /tubes/n5_4 -> /tubes/n2_3
- J6 pad 6: /tubes/n5_5 -> /tubes/n2_2
- J6 pad 7: /tubes/n5_6 -> /tubes/n2_1
- J6 pad 8: /tubes/n5_7 -> /tubes/n2_0
- J6 pad 9: /tubes/n5_8 -> /tubes/n2_9
- R10 pad 2: Net-(NE2-Pad1) -> Net-(NE3-Pad1)
- R11 pad 2: Net-(R11-Pad2) -> Net-(NE4-Pad1)
- R13 pad 2: Net-(NE3-Pad1) -> Net-(R13-Pad2)
- R2 pad 1: Net-(R2-Pad1) -> +3V3
- R2 pad 2: Net-(Q1-Pad2) -> Net-(R2-Pad2)
- R3 pad 1: +3V3 -> Net-(R2-Pad2)
- R3 pad 2: Net-(R3-Pad2) -> GND
- R4 pad 1: Net-(R3-Pad2) -> Net-(R4-Pad1)
- R4 pad 2: GND -> HT
- R5 pad 2: /vHtMon -> Net-(R5-Pad2)
- R6 pad 1: /vHtMon -> HT
- R6 pad 2: GND -> Net-(NE1-Pad1)
- R7 pad 1: Net-(R7-Pad1) -> HT
- R7 pad 2: HT -> Net-(NE2-Pad1)
- R9 pad 2: Net-(NE1-Pad1) -> Net-(R9-Pad2)
- U1 pad 1: Net-(R3-Pad2) -> Net-(U1-Pad1)
- U1 pad 2: +3V3 -> /tubes/clk
- U1 pad 3: +12V -> Net-(U1-Pad3)
- U1 pad 4: +3V3 -> GND
- U10 pad 1: Net-(R11-Pad2) -> Net-(R8-Pad2)
- U11 pad 1: Net-(R12-Pad2) -> Net-(R9-Pad2)
- U12 pad 1: Net-(R15-Pad2) -> Net-(R12-Pad2)
- U13 pad 1: Net-(R16-Pad2) -> Net-(R13-Pad2)
- U3 pad 10: Net-(Q4-Pad1) -> Net-(U1-Pad6)
- U3 pad 11: Net-(Q3-Pad1) -> Net-(U1-Pad3)
- U3 pad 12: Net-(Q2-Pad1) -> Net-(U1-Pad1)
- U3 pad 24: Net-(R2-Pad1) -> Net-(U3-Pad24)
- U3 pad 8: /vHtMon -> Net-(U3-Pad8)
- U6 pad 1: Net-(R7-Pad1) -> Net-(R4-Pad1)
- U7 pad 27: +12V -> +5V
- U7 pad 30: +12V -> +5V
- U7 pad 33: +12V -> +5V
- U8 pad 27: +12V -> +5V
- U8 pad 30: +12V -> +5V
- U8 pad 33: +12V -> +5V
- U9 pad 1: Net-(R8-Pad2) -> Net-(R5-Pad2)
Routing:
- net /tubes/clk: track 0.00 -> 71.0 mm, vias 0 -> 2
- net Net-(U7-Pad23): track 0.00 -> 56.7 mm, vias 0 -> 2
- net /tubes/nLatch: track 0.00 -> 55.8 mm, vias 0 -> 2
- net Net-(U1-Pad6): track 0.00 -> 53.9 mm, vias 0 -> 1
- net Net-(R15-Pad2): track 48.9 -> 0.00 mm, vias 2 -> 0
- net Net-(R12-Pad2): track 42.4 -> 91.3 mm, vias 2 -> 4
- net Net-(U1-Pad3): track 0.00 -> 48.6 mm, vias 0 -> 1
- net Net-(R16-Pad2): track 45.3 -> 0.00 mm, vias 2 -> 0
- net Net-(R13-Pad2): track 0.00 -> 45.3 mm, vias 0 -> 2
- net Net-(U1-Pad1): track 0.00 -> 42.3 mm, vias 0 -> 1
- net /rstBtn: track 0.00 -> 37.1 mm, vias 0 -> 1
- net /progFlag: track 0.00 -> 23.7 mm, vias 0 -> 1
- net GND: track 0.00 -> 14.5 mm, vias 19 -> 22
- net Net-(P1-Pad4): track 0.00 -> 13.6 mm, vias 0 -> 1
- net +3V3: track 0.00 -> 12.5 mm, vias 0 -> 1
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
Commit message: done, done done done
Parts:
- removed the R4 at (91.8, 81.6)
- removed the R5 at (77.2, 68.3)
- removed the R6 at (54.8, 67.6)
- added C7: 1u, Capacitor_SMD:C_0805_2012Metric, F.Cu at (53.9, 108.9)
- added J7: Conn_01x04, Connector_PinHeader_2.54mm:PinHeader_1x04_P2.54mm_Vertical, F.Cu at (56.5, 98.7)
- added R10: 10k, Resistor_SMD:R_0805_2012Metric, B.Cu at (130.1, 53.0)
- added R12: 10k, Resistor_SMD:R_0805_2012Metric, B.Cu at (135.2, 53.0)
- added R8: 10k, Resistor_SMD:R_0805_2012Metric, B.Cu at (74.3, 23.8)
- added U14: SN74LVC2G17, Package_TO_SOT_SMD:SOT-363_SC-70-6, B.Cu at (53.9, 108.9)
- C3, C4, C6, R2, R3: moved to F.Cu
- J1, J2: moved to B.Cu
- U1: value 74LVC3G34DP -> SN74LVC2G17; footprint Package_SO:VSSOP-8_2.4x2.1mm_P0.5mm -> Package_TO_SOT_SMD:SOT-363_SC-70-6
- moved C3 100.4 mm to (147.9, 131.7)
- moved U2 92.8 mm to (147.9, 124.1), turned to 0 degrees
- moved C6 86.0 mm to (121.5, 125.4), turned to 180 degrees
- moved C4 84.9 mm to (142.8, 114.0)
- moved R2 83.4 mm to (142.8, 116.5), turned to 180 degrees
- moved R3 62.4 mm to (137.8, 116.5), turned to 180 degrees
- moved R11 58.5 mm to (125.1, 52.7), turned to 90 degrees
- moved C5 36.5 mm to (73.7, 105.6), turned to 0 degrees
- moved J2 29.4 mm to (94.6, 105.1), turned to 90 degrees
- moved J1 25.6 mm to (140.3, 131.7), turned to 270 degrees
- moved R13 10.2 mm to (140.3, 53.0)
- turned C1 to 0 degrees
- renumbered R7 to R4, R8 to R5, R9 to R6, R10 to R7, R12 to R9
Connections:
- R4 pad 1: HT -> Net-(R4-Pad1)
- R4 pad 2: Net-(NE2-Pad1) -> HT
- R5 pad 2: Net-(R8-Pad2) -> Net-(R5-Pad2)
- R6 pad 2: Net-(R9-Pad2) -> Net-(NE1-Pad1)
- R7 pad 2: Net-(NE3-Pad1) -> Net-(NE2-Pad1)
- R9 pad 2: Net-(R12-Pad2) -> Net-(R9-Pad2)
- U1 pad 2: /tubes/clk -> GND
- U1 pad 4: GND -> /tubes/dat
- U1 pad 5: /tubes/dat -> +5V
- U1 pad 6: Net-(U1-Pad6) -> /tubes/nLatch
- U3 pad 10: Net-(U1-Pad6) -> Net-(U14-Pad1)
Routing:
- net +5V: track 3.05 -> 210.7 mm, vias 1 -> 8
- net +3V3: track 12.5 -> 126.3 mm
- net Net-(U1-Pad6): track 53.9 -> 0.00 mm, vias 1 -> 0
- net Net-(R9-Pad2): track 0.00 -> 42.4 mm, vias 0 -> 2
- net Net-(R12-Pad2): track 91.3 -> 48.9 mm, vias 4 -> 2
- net Net-(J7-Pad4): track 0.00 -> 40.5 mm, vias 0 -> 2
- net /tubes/clk: track 71.0 -> 106.4 mm, vias 2 -> 3
- net Net-(U14-Pad1): track 0.00 -> 29.7 mm, vias 0 -> 1
- net Net-(U14-Pad3): track 0.00 -> 26.8 mm, vias 0 -> 1
- net GND: track 14.5 -> 38.5 mm, vias 22 -> 38
- net Net-(R11-Pad2): track 20.0 -> 0.00 mm
- net Net-(R7-Pad1): track 17.7 -> 0.00 mm
- net Net-(R4-Pad1): track 0.00 -> 17.7 mm
- net HT: track 125.1 -> 139.0 mm
- net Net-(R8-Pad2): track 6.98 -> 20.0 mm
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- added copper zone on F.Cu, net +3V3
