File: pcb/nixie/nixie.kicad_pcb (KiCad board)
At the start: 2 copper layers, 144 x 116 mm, 58 parts, among them J1 Conn_01x02, J2 Conn_01x02, J3 Conn_01x32, J4 Conn_01x32, J5 Conn_01x32, J6 Conn_01x32, J7 Conn_01x04, P1 TTL_232R_3V3, Q1 BSS138, Q2 BSS138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

Commit message: Minor imprpvements
Parts:
- J7: moved to B.Cu
- turned J7 to 270 degrees
Routing:
- net Net-(Q2-Pad2): track 40.7 -> 38.7 mm
- net Net-(Q1-Pad2): track 39.6 -> 40.6 mm
- net +3V3: track 187.9 -> 188.7 mm
